File: Electronics/PCB_Design/ATEx_2016/ATEx_2016.brd (EAGLE design)
At the start: 127 x 63.2 mm, 43 parts, among them IC2 REG1117, IC3 DS1307, IC5 ON M74VHC1GT125DT1G, J1 POWER_JACKPTH, J2 J5MM, M1 HX1, Q1 32.768, Q2 8/16/20MHz, U1 BMP180, U3 LSM9DS1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

Commit message: Updates
Parts:
- added JP13: (no value), SparkFun-Connectors:1X03
Connections:
- new net P9_31B: JP13.1
- net 5V: now also JP13.2
- net GND: now also JP13.3
- net I2C1_SCL: no longer R2.1, U1.5, U3.2
- net I2C1_SDA: no longer R1.1, U1.6, U3.4
- net I2C2_SCL: now also R2.1, U1.5, U3.2
- net I2C2_SDA: now also R1.1, U1.6, U3.4
Changed lines of the file:
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@@
 <attribute name="PROD_ID" value="RES-00824" x="-2.54" y="-59.69" size="1.778" layer="27" display="off"/>
 </element>
+<element name="JP13" library="SparkFun-Connectors" package="1X03" value="" x="-2.54" y="-58.42"/>
 </elements>
 <signals>
@@
 <contactref element="C13" pad="2"/>
 <contactref element="C18" pad="2"/>
+<contactref element="JP13" pad="3"/>
 <wire x1="89.85" y1="71.1" x2="97.79" y2="81.28" width="0" layer="19" extent="1-1"/>
 <wire x1="87.95" y1="71.1" x2="89.85" y2="71.1" width="0" layer="19" extent="1-1"/>
@@
 <wire x1="2.12" y1="-44.45" x2="-1.69" y2="-44.45" width="0" layer="19" extent="1-1"/>
 <wire x1="2.12" y1="-40.64" x2="-1.69" y2="-40.64" width="0" layer="19" extent="1-1"/>
+<wire x1="2.54" y1="-58.42" x2="2.12" y2="-44.45" width="0" layer="19" extent="1-1"/>
 </signal>
 <signal name="3.3V">
@@
 <contactref element="BB1" pad="P9.6"/>
 <contactref element="BB1" pad="P9.5"/>
+<contactref element="JP13" pad="2"/>
 <wire x1="107.55" y1="52.8574" x2="109.95" y2="61.4426" width="0" layer="19" extent="1-1"/>
 <wire x1="86.36" y1="81.28" x2="109.95" y2="61.4426" width="0" layer="19" extent="1-1"/>
@@
 <wire x1="24.13" y1="73.025" x2="15.24" y2="60.96" width="0" layer="19" extent="1-1"/>
 <wire x1="24.13" y1="75.565" x2="24.13" y2="73.025" width="0" layer="19" extent="1-1"/>
+<wire x1="0" y1="-58.42" x2="41.91" y2="39.37" width="0" layer="19" extent="1-1"/>
 </signal>
 <signal name="I2C2_SDA">
 <contactref element="IC3" pad="5"/>
 <contactref element="BB1" pad="P9.20"/>
+<contactref element="U3" pad="4"/>
+<contactref element="U1" pad="6"/>
+<contactref element="R1" pad="1"/>
 <wire x1="15.24" y1="68.58" x2="41.91" y2="73.025" width="0" layer="19" extent="1-1"/>
+<wire x1="-1.04" y1="13.79" x2="15.24" y2="68.58" width="0" layer="19" extent="1-1"/>
+<wire x1="0.42" y1="5.08" x2="-1.04" y2="13.79" width="0" layer="19" extent="1-1"/>
+<wire x1="-4.015" y1="-35.775" x2="0.42" y2="5.08" width="0" layer="19" extent="1-1"/>
 </signal>
 <signal name="I2C2_SCL">
 <contactref element="IC3" pad="6"/>
 <contactref element="BB1" pad="P9.19"/>
+<contactref element="U3" pad="2"/>
+<contactref element="U1" pad="5"/>
+<contactref element="R2" pad="1"/>
 <wire x1="15.24" y1="66.04" x2="41.91" y2="75.565" width="0" layer="19" extent="1-1"/>
+<wire x1="-2.54" y1="13.79" x2="15.24" y2="66.04" width="0" layer="19" extent="1-1"/>
+<wire x1="4.23" y1="5.08" x2="-2.54" y2="13.79" width="0" layer="19" extent="1-1"/>
+<wire x1="-4.015" y1="-34.915" x2="4.23" y2="5.08" width="0" layer="19" extent="1-1"/>
 </signal>
 <signal name="3VOLT">
@@
 <signal name="I2C1_SCL">
 <contactref element="BB1" pad="P9.17"/>
-<contactref element="U1" pad="5"/>
-<contactref element="R2" pad="1"/>
-<contactref element="U3" pad="2"/>
-<wire x1="-2.54" y1="13.79" x2="39.37" y2="75.565" width="0" layer="19" extent="1-1"/>
-<wire x1="4.23" y1="5.08" x2="-2.54" y2="13.79" width="0" layer="19" extent="1-1"/>
-<wire x1="-4.015" y1="-34.915" x2="4.23" y2="5.08" width="0" layer="19" extent="1-1"/>
 </signal>
 <signal name="N$62">
@@
 <signal name="I2C1_SDA">
 <contactref element="BB1" pad="P9.18"/>
-<contactref element="U1" pad="6"/>
-<contactref element="R1" pad="1"/>
-<contactref element="U3" pad="4"/>
-<wire x1="-1.04" y1="13.79" x2="39.37" y2="73.025" width="0" layer="19" extent="1-1"/>
-<wire x1="0.42" y1="5.08" x2="-1.04" y2="13.79" width="0" layer="19" extent="1-1"/>
-<wire x1="-4.015" y1="-35.775" x2="0.42" y2="5.08" width="0" layer="19" extent="1-1"/>
 </signal>
 <signal name="N$79">
@@
 <wire x1="-3.615" y1="-34.335" x2="0.42" y2="-40.64" width="0" layer="19" extent="1-1"/>
 </signal>
+<signal name="P9_31B">
+<contactref element="JP13" pad="1"/>
+</signal>
 </signals>

Commit message: Added components
Parts:
- added J3, J4: 2X6 FEMALE, SparkFun-Connectors:2X6
Other:
- board size 127 x 63.2 mm -> 100.3 x 100 mm
Changed lines of the file:
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@@
 <layer number="112" name="tSilk" color="7" fill="1" visible="yes" active="yes"/>
 <layer number="113" name="IDFDebug" color="4" fill="1" visible="yes" active="yes"/>
+<layer number="114" name="Badge_Outline" color="7" fill="1" visible="yes" active="yes"/>
+<layer number="115" name="ReferenceISLANDS" color="7" fill="1" visible="yes" active="yes"/>
 <layer number="116" name="Patch_BOT" color="9" fill="4" visible="yes" active="yes"/>
 <layer number="118" name="Rect_Pads" color="7" fill="1" visible="yes" active="yes"/>
@@
 <board>
 <plain>
-<wire x1="0" y1="20.32" x2="126.98" y2="20.32" width="0" layer="20"/>
-<wire x1="126.98" y1="20.32" x2="126.98" y2="83.49" width="0" layer="20"/>
-<wire x1="126.98" y1="83.49" x2="0" y2="83.49" width="0" layer="20"/>
-<wire x1="0" y1="83.49" x2="0" y2="20.32" width="0" layer="20"/>
+<wire x1="0" y1="0" x2="100.31" y2="0" width="0" layer="20"/>
+<wire x1="100.31" y1="0" x2="100.31" y2="100" width="0" layer="20"/>
+<wire x1="100.31" y1="100" x2="0" y2="100" width="0" layer="20"/>
+<wire x1="0" y1="100" x2="0" y2="0" width="0" layer="20"/>
 </plain>
 <attributes>
@@
 </element>
 <element name="JP13" library="SparkFun-Connectors" package="1X03" value="" x="-2.54" y="-58.42"/>
+<element name="J3" library="SparkFun-Connectors" package="2X6" value="2X6 FEMALE" x="-2.54" y="-66.04">
+<attribute name="PROD_ID" value="CONN-12423" x="-2.54" y="-66.04" size="1.778" layer="27" display="off"/>
+</element>
+<element name="J4" library="SparkFun-Connectors" package="2X6" value="2X6 FEMALE" x="-2.54" y="-76.2">
+<attribute name="PROD_ID" value="CONN-12423" x="-2.54" y="-76.2" size="1.778" layer="27" display="off"/>
+</element>
 </elements>
 <signals>

Commit message: Finalized PCB design
Parts:
- removed C15, C16: 10uF, rcl:E2,5-5
- removed X2: BU-SMA-V, con-coax:BU-SMA-V
- added C10, C5: 10uF, SparkFun:EIA3216
- added JP1: JUMPER-PAD-2-NC_BY_TRACE, SparkFun-Passives:PAD-JUMPER-2-NC_BY_TRACE_YES_SILK
- added X1: BU-SMA-V, con-coax:BU-SMA-V
- BB1: value BBH2 -> BBH1; device logic-supply:BB_CAPE_TOP -> logic-supply:BB_CAPE
- C4: device adafruit:C1206 -> adafruit:C0603
- C7, C8: device SparkFun-Passives:1206 -> SparkFun-Passives:0603-CAP
- R14, R15: value 4.7k -> 220; device logic-supply:R0805 -> logic-supply:R0603
- R9: device SparkFun-Passives:1206 -> SparkFun-Passives:0603-RES
- moved JP13 149.9 mm to (40.6, 85.1)
- moved R10 121.6 mm to (59.7, 58.4)
- moved R8 121.3 mm to (59.7, 55.9)
- moved R12 120.9 mm to (61.6, 52.7)
- moved R11 119.5 mm to (57.1, 51.4)
- moved J4 117.0 mm to (3.81, 40.6), turned to 270 degrees
- moved C18 115.3 mm to (50.8, 59.7), turned to 270 degrees
- moved C17 113.6 mm to (48.3, 57.1), turned to 90 degrees
- moved C12 110.3 mm to (55.9, 63.5), turned to 270 degrees
- moved U3 109.2 mm to (55.2, 57.1), turned to 90 degrees
- moved C13 108.2 mm to (53.3, 52.1), turned to 270 degrees
- moved C14 105.9 mm to (48.9, 54.0), turned to 180 degrees
- moved J3 90.4 mm to (3.81, 24.1), turned to 270 degrees
- moved BAT 81.7 mm to (82.5, 83.8), turned to 270 degrees
- moved C2 72.0 mm to (44.5, 59.7)
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Connections:
- net N$68 renamed AIN1
- net N$69 renamed AIN3
- net N$70 renamed AIN5
- removed net N$41: BB1.P8.19
- removed net N$51: BB1.P9.39
- removed net N$52: BB1.P9.37
- removed net N$53: BB1.P9.35
- removed net N$54: BB1.P9.33
- removed net N$63: BB1.P9.13
- removed net N$64: BB1.P9.11
- removed net P9_31B: JP13.1
- new net +3V3: C12.1, C13.1, C18.1, JP1.1, U3.1, U3.22, U3.23, U3.3
- new net AIN0: BB1.P9.39, J3.2
- new net AIN2: BB1.P9.37, J3.11
- new net AIN4: BB1.P9.33, J4.11
- new net AIN6: BB1.P9.35, J4.2
- new net N$14: IC5.3
- new net P8_19: BB1.P8.19, JP13.1
- new net UART4_RX: BB1.P9.11, J3.7
- new net UART4_TX: BB1.P9.13, J3.9
- net 3.3V: now also C5.A, J3.1, J4.1, JP1.2; no longer C12.1, C13.1, C15.+, C18.1, U3.1, U3.22, U3.23, U3.3
- net 5V: now also C10.A; no longer C16.+
- net GND: now also C10.C, C5.C, J3.12, J4.12, X1.2, X1.3, X1.4, X1.5; no longer C15.-, C16.-, IC5.3, X2.2, X2.3, X2.4, X2.5
- net I2C1_SCL: now also J3.5, J4.5
- net I2C1_SDA: now also J3.3, J4.3
- net RFOUT: now also X1.1; no longer X2.1
- net UART2_RX: now also J4.7
- net UART2_TX: now also J4.9
Routing:
- net 5V: track 0.00 -> 248.7 mm
- net GND: track 0.00 -> 163.5 mm
- net AIN4: track 0.00 -> 82.5 mm
- net AIN2: track 0.00 -> 77.7 mm
- net I2C2_SCL: track 0.00 -> 76.0 mm
- net AIN0: track 0.00 -> 72.7 mm
- net RXI: track 0.00 -> 69.2 mm
- net AIN6: track 0.00 -> 60.8 mm, vias 0 -> 1
- net I2C1_SDA: track 0.00 -> 60.1 mm
- net I2C2_SDA: track 0.00 -> 59.9 mm, vias 0 -> 1
- net I2C1_SCL: track 0.00 -> 59.9 mm
- net UART2_RX: track 0.00 -> 56.1 mm
- net UART4_TX: track 0.00 -> 54.4 mm, vias 0 -> 1
- net UART4_RX: track 0.00 -> 53.2 mm
- net UART2_TX: track 0.00 -> 50.6 mm
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- added copper zone on layer 15, net 3.3V
- added copper zone on layer 2, net GND
Other:
- board size 100.3 x 100 mm -> 100.3 x 100.3 mm
