File: Electronics/PCB_Design/ATEx_2016/ATEx_2016.sch (EAGLE design)
At the start: 43 parts, among them IC2 REG1117, IC3 DS1307, IC5 ON M74VHC1GT125DT1G, J1 POWER_JACKPTH, J2 J5MM, M1 HX1, Q1 32.768, Q2 8/16/20MHz, U1 BMP180, U3 LSM9DS1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

Commit message: Updates
Parts:
- added JP13: (no value), SparkFun-Connectors:M03PTH
Connections:
- new net P9_31B: JP13.1
- net 5V: now also JP13.2
- net GND: now also JP13.3
- net I2C1_SCL: no longer R2.1, U1.SCL, U3.SCL/SPC
- net I2C1_SDA: no longer R1.1, U1.SDA, U3.SDA/SDI/SDO
- net I2C2_SCL: now also R2.1, U1.SCL, U3.SCL/SPC
- net I2C2_SDA: now also R1.1, U1.SDA, U3.SDA/SDI/SDO

Commit message: Added components
Parts:
- added J3, J4: 2X6 FEMALE, SparkFun-Connectors:M06X2PTH_FEMALE
Changed lines of the file:
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@@
 <layer number="112" name="tSilk" color="7" fill="1" visible="yes" active="yes"/>
 <layer number="113" name="IDFDebug" color="4" fill="1" visible="yes" active="yes"/>
+<layer number="114" name="Badge_Outline" color="7" fill="1" visible="yes" active="yes"/>
+<layer number="115" name="ReferenceISLANDS" color="7" fill="1" visible="yes" active="yes"/>
 <layer number="116" name="Patch_BOT" color="9" fill="4" visible="yes" active="yes"/>
 <layer number="118" name="Rect_Pads" color="7" fill="1" visible="yes" active="yes"/>
@@
 <part name="GND14" library="supply1" deviceset="GND" device=""/>
 <part name="U$13" library="SparkFun-Aesthetics" deviceset="5V" device=""/>
+<part name="J3" library="SparkFun-Connectors" deviceset="M06X2" device="PTH_FEMALE" value="2X6 FEMALE"/>
+<part name="J4" library="SparkFun-Connectors" deviceset="M06X2" device="PTH_FEMALE" value="2X6 FEMALE"/>
 </parts>
 <sheets>
 <sheet>
 <plain>
-<wire x1="-190.5" y1="53.34" x2="-5.08" y2="50.8" width="0.1524" layer="97" style="shortdash"/>
-<wire x1="-5.08" y1="50.8" x2="-7.62" y2="-129.54" width="0.1524" layer="97" style="shortdash"/>
+<wire x1="-190.5" y1="53.34" x2="-7.62" y2="53.34" width="0.1524" layer="97" style="shortdash"/>
+<wire x1="-7.62" y1="53.34" x2="-7.62" y2="-129.54" width="0.1524" layer="97" style="shortdash"/>
 <text x="-182.88" y="43.18" size="2.54" layer="97" font="vector">BeagleBone Headers</text>
 <text x="167.64" y="-106.68" size="2.54" layer="97" font="vector">2</text>
@@
 </instance>
 <instance part="U$13" gate="G$1" x="-17.78" y="35.56" rot="R270"/>
+<instance part="J3" gate="G$1" x="-35.56" y="2.54"/>
+<instance part="J4" gate="G$1" x="-35.56" y="-25.4"/>
 </instances>
 <busses>

Commit message: Finalized PCB design
Parts:
- removed C15, C16: 10uF, rcl:CPOL-EUE2.5-5
- added C10, C5: 10uF, SparkFun:CAP_POL1206
- added JP1: JUMPER-PAD-2-NC_BY_TRACE, SparkFun-Passives:JUMPER-PAD-2-NC_BY_TRACE
- BB1: value BBH2 -> BBH1; device logic-supply:BBH2 -> logic-supply:BBH1
- C4: device adafruit:C-USC1206 -> adafruit:C-USC0603
- C7, C8: device SparkFun-Passives:CAP1206 -> SparkFun-Passives:CAP0603-CAP
- R14, R15: value 4.7k -> 220; device logic-supply:R0805 -> logic-supply:R0603
- R9: device SparkFun-Passives:RESISTOR1206 -> SparkFun-Passives:RESISTOR0603-RES
- renumbered X2 to X1
Connections:
- net N$68 renamed AIN1
- net N$69 renamed AIN3
- net N$70 renamed AIN5
- removed net N$41: BB1P8.PWM2A/GPIO0_22
- removed net N$51: BB1P9.AIN0
- removed net N$52: BB1P9.AIN2
- removed net N$53: BB1P9.AIN6
- removed net N$54: BB1P9.AIN4
- removed net N$63: BB1P9.SERIAL4_TX/GPIO0_31
- removed net N$64: BB1P9.SERIAL4_RX/GPIO0_30
- removed net P9_31B: JP13.1
- new net +3V3: C12.1, C13.1, C18.1, JP1.1, U3.VDD, U3.VDDIO
- new net AIN0: BB1P9.AIN0, J3.2
- new net AIN2: BB1P9.AIN2, J3.11
- new net AIN4: BB1P9.AIN4, J4.11
- new net AIN6: BB1P9.AIN6, J4.2
- new net N$14: IC5P.GND
- new net P8_19: BB1P8.PWM2A/GPIO0_22, JP13.1
- new net UART4_RX: BB1P9.SERIAL4_RX/GPIO0_30, J3.7
- new net UART4_TX: BB1P9.SERIAL4_TX/GPIO0_31, J3.9
- net 3.3V: now also C5.+, J3.1, J4.1, JP1.2; no longer C12.1, C13.1, C15.+, C18.1, U3.VDD, U3.VDDIO
- net 5V: now also C10.+; no longer C16.+
- net GND: now also C10.-, C5.-, J3.12, J4.12; no longer C15.-, C16.-, IC5P.GND
- net I2C1_SCL: now also J3.5, J4.5
- net I2C1_SDA: now also J3.3, J4.3
- net UART2_RX: now also J4.7
- net UART2_TX: now also J4.9
Other:
- moved on the sheet: IC2
